Commit message: fix macros path

File: cartographer_config/f110_description/urdf/macros.xacro (robot description, xacro)
@@ -41,5 +41,5 @@
   <origin xyz="0 0 0" rpy="0 0 0" />
   <geometry>
-    <mesh filename="package://racecar_description/meshes/chassis.STL" />
+    <mesh filename="package://f110_description/meshes/chassis.STL" />
   </geometry>
 </xacro:macro>
@@ -47,5 +47,5 @@
   <origin xyz="0 0 0" rpy="0 0 0" />
   <geometry>
-    <mesh filename="package://racecar_description/meshes/left_rear_wheel.STL" />
+    <mesh filename="package://f110_description/meshes/left_rear_wheel.STL" />
   </geometry>
 </xacro:macro>
@@ -53,5 +53,5 @@
   <origin xyz="0 0 0" rpy="0 0 0" />
   <geometry>
-    <mesh filename="package://racecar_description/meshes/right_rear_wheel.STL" />
+    <mesh filename="package://f110_description/meshes/right_rear_wheel.STL" />
   </geometry>
 </xacro:macro>
@@ -59,5 +59,5 @@
   <origin xyz="0 0 0" rpy="0 0 0" />
   <geometry>
-    <mesh filename="package://racecar_description/meshes/left_front_wheel.STL" />
+    <mesh filename="package://f110_description/meshes/left_front_wheel.STL" />
   </geometry>
 </xacro:macro>
@@ -65,5 +65,5 @@
   <origin xyz="0 0 0" rpy="0 0 0" />
   <geometry>
-    <mesh filename="package://racecar_description/meshes/right_front_wheel.STL" />
+    <mesh filename="package://f110_description/meshes/right_front_wheel.STL" />
   </geometry>
 </xacro:macro>
@@ -71,5 +71,5 @@
   <origin xyz="0 0 0" rpy="0 0 0" />
   <geometry>
-    <mesh filename="package://racecar_description/meshes/left_steering_hinge.STL" />
+    <mesh filename="package://f110_description/meshes/left_steering_hinge.STL" />
   </geometry>
 </xacro:macro>
@@ -77,5 +77,5 @@
   <origin xyz="0 0 0" rpy="0 0 0" />
   <geometry>
-    <mesh filename="package://racecar_description/meshes/right_steering_hinge.STL" />
+    <mesh filename="package://f110_description/meshes/right_steering_hinge.STL" />
   </geometry>
 </xacro:macro>
